File: PCB_panel/PCB_panel.kicad_pcb (KiCad board)
At the start: 2 copper layers, 100 x 80 mm, 28 parts, among them J1 Conn_01x05_Pin, J10 OLed screen, J2 Conn_01x05_Pin, J3 Conn_01x05_Pin, SW10 SW_Push, SW11 SW_HDMI, SW12 SW_USB, SW2 SW_Push, SW3 SW_Push, SW4 SW_Push, SW5 SW_Push, SW6 SW_Push, SW7 SW_Push, SW8 SW_Push, SW9 SW_Push, U1 COM-09032

Commit message: update pcb
Parts:
- removed R2, R3: 4.7k, Resistor_THT:R_Axial_DIN0207_L6.3mm_D2.5mm_P10.16mm_Horizontal
- D1, D2, D3, D4, D5, D6, D7, D8, D9, R1: moved to B.Cu
- J1: value Conn_01x05_Pin -> Conn 1; moved to B.Cu
- J2: value Conn_01x05_Pin -> Conn 2; moved to B.Cu
- J3: value Conn_01x05_Pin -> Conn 3; moved to B.Cu
- U1: value COM-09032 -> Joystick
- renumbered SW2 to SW1, SW12 to SW10, SW3 to SW2, SW4 to SW3, SW5 to SW4, SW6 to SW5, SW7 to SW6, SW8 to SW7, SW9 to SW8, SW10 to SW9, J10 to U2
Routing:
- net +3.3V: track 116.5 -> 100.9 mm
- net /SCL: track 69.2 -> 53.6 mm
- net /SDA: track 76.1 -> 65.3 mm
- net /Ligne_2: track 74.7 -> 75.9 mm
Other:
- board text added: "Designed in Roanne"
- board text added: "V1.3.7"
- board text removed: "Made in Roanne"
- board text removed: "V1.3.1"
