File: PCB_panel/PCB_panel.kicad_sch (KiCad schematic)
At the start: 28 parts, among them J1 Conn_01x05_Pin, J10 OLed screen, J2 Conn_01x05_Pin, J3 Conn_01x05_Pin, SW10 SW_Push, SW11 SW_HDMI, SW12 SW_USB, SW2 SW_Push, SW3 SW_Push, SW4 SW_Push, SW5 SW_Push, SW6 SW_Push, SW7 SW_Push, SW8 SW_Push, SW9 SW_Push, U1 COM-09032

Commit message: update pcb
Parts:
- removed R2, R3: 4.7k, Resistor_THT:R_Axial_DIN0207_L6.3mm_D2.5mm_P10.16mm_Horizontal, symbol Device:R
- removed SW2: SW_Push, Library:PVA1 OA H1 1.2N V2, symbol Switch:SW_Push_45deg
- added SW1: SW_Push, Library:PVA1 OA H1 1.2N V2, symbol Switch:SW_Push_45deg
- J1: value Conn_01x05_Pin -> Conn 1
- J2: value Conn_01x05_Pin -> Conn 2
- J3: value Conn_01x05_Pin -> Conn 3
- U1: value COM-09032 -> Joystick
- renumbered SW12 to SW10, SW3 to SW2, SW4 to SW3, SW5 to SW4, SW6 to SW5, SW7 to SW6, SW8 to SW7, SW9 to SW8, SW10 to SW9, J10 to U2
Connections:
- net Col_0: now also SW1.1
- net at D1.2 (A): now also SW1.2
Other:
- note added: "PIN TO PCB CONTROLEUR"
- moved on the sheet: D1, D2, D3, D4, D5, D6, D7, D8, D9, J1, J2, J3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
